File: Battery_Charger.kicad_pcb (KiCad board)
At the start: 2 copper layers, 16.5 x 25.6 mm, 9 parts, among them J1 USB_B_Micro, J2 Conn_01x02, U1 MCP73831-2-OT

Commit message: Removed copper fill....
Routing:
- net GND: track 20.1 -> 42.5 mm
- removed copper zone on F.Cu, net GND
Changed lines of the file:
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@@
+	)
+	(segment
+		(start 147.475 83.405)
+		(end 147.205 83.675)
+		(width 0.25)
+		(layer "F.Cu")
+		(net 2)
+	)
+	(segment
+		(start 141.23 86.5675)
+		(end 142.8525 84.945)
+		(width 0.25)
+		(layer "F.Cu")
+		(net 2)
+	)
+	(segment
+		(start 147.475 78.9875)
+		(end 147.475 83.405)
+		(width 0.25)
+		(layer "F.Cu")
+		(net 2)
+	)
+	(segment
+		(start 144.6825 75.5625)
+		(end 144.6825 76.195)
+		(width 0.25)
+		(layer "F.Cu")
+		(net 2)
 	)
 	(segment
@@
 	)
 	(segment
+		(start 141.23 89.105)
+		(end 141.23 86.5675)
+		(width 0.25)
+		(layer "F.Cu")
+		(net 2)
+	)
+	(segment
 		(start 138.235 73.535)
 		(end 138.545 73.225)
@@
 	)
 	(segment
+		(start 145.575 83.675)
+		(end 144.1225 83.675)
+		(width 0.25)
+		(layer "F.Cu")
+		(net 2)
+	)
+	(segment
 		(start 140.845 70.525)
 		(end 138.845 70.525)
@@
 	)
 	(segment
+		(start 142.345 73.225)
+		(end 144.6825 75.5625)
+		(width 0.25)
+		(layer "F.Cu")
+		(net 2)
+	)
+	(segment
 		(start 137.655 73.535)
 		(end 138.235 73.535)
@@
 	)
 	(segment
+		(start 144.6825 76.195)
+		(end 147.475 78.9875)
+		(width 0.25)
+		(layer "F.Cu")
+		(net 2)
+	)
+	(segment
+		(start 144.1225 83.675)
+		(end 142.8525 84.945)
+		(width 0.25)
+		(layer "F.Cu")
+		(net 2)
+	)
+	(segment
 		(start 141.19 81.375882)
 		(end 141.19 83.2825)
@@
 	)
 	(segment
+		(start 147.205 83.675)
+		(end 145.575 83.675)
+		(width 0.25)
+		(layer "F.Cu")
+		(net 2)
+	)
+	(segment
 		(start 141.19 83.2825)
 		(end 142.8525 84.945)
@@
 	)
 	(segment
-		(start 138.34 80.597501)
-		(end 138.34 84.82)
+		(start 137.655 85.505)
+		(end 137.395 85.765)
+		(width 0.25)
+		(layer "F.Cu")
+		(net 8)
+	)
+	(segment
+		(start 139.9525 79.6475)
+		(end 138.6875 79.6475)
+		(width 0.25)
+		(layer "F.Cu")
+		(net 8)
+	)
+	(segment
+		(start 138.6875 79.6475)
+		(end 137.655 80.68)
+		(width 0.25)
+		(layer "F.Cu")
+		(net 8)
+	)
+	(segment
+		(start 137.655 80.68)
+		(end 137.655 85.505)
 		(width 0.25)
 		(layer "F.Cu")
@@
 	)
 	(segment
-		(start 139.9525 79.6475)
-		(end 139.290001 79.6475)
-		(width 0.25)
-		(layer "F.Cu")
-		(net 8)
-	)
-	(segment
-		(start 139.290001 79.6475)
-		(end 138.34 80.597501)
-		(width 0.25)
-		(layer "F.Cu")
-		(net 8)
-	)
-	(segment
-		(start 138.34 84.82)
-		(end 137.395 85.765)
-		(width 0.25)
-		(layer "F.Cu")
-		(net 8)
-	)
-	(segment
 		(start 143.4 79.815)
 		(end 143.2325 79.6475)
@@
 		(net 9)
 	)
-	(zone
-		(net 2)
-		(net_name "GND")
-		(layer "F.Cu")
-		(hatch edge 0.5)
-		(connect_pads
-			(clearance 0.5)
-		)
-		(min_thickness 0.25)
-		(filled_areas_thickness no)
-		(fill yes
-			(thermal_gap 0.5)
-			(thermal_bridge_width 0.5)
-		)
-		(polygon
-			(pts
-				(xy 132.33 68.565) (xy 132.505 90.52) (xy 148.335 90.52) (xy 148.165 68.575)
-			)
-		)
-	)
 )

Commit message: Added copper fill
Routing:
- added copper zone on F.Cu, net GND
Changed lines of the file:
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@@
 		(net 9)
 	)
+	(zone
+		(net 2)
+		(net_name "GND")
+		(layer "F.Cu")
+		(hatch edge 0.5)
+		(connect_pads
+			(clearance 0.5)
+		)
+		(min_thickness 0.25)
+		(filled_areas_thickness no)
+		(fill yes
+			(thermal_gap 0.5)
+			(thermal_bridge_width 0.5)
+		)
+		(polygon
+			(pts
+				(xy 132.385 68.915) (xy 148.445 69.055) (xy 148.505 94.3) (xy 132.365 94.265) (xy 132.4 69.305)
+			)
+		)
+	)
 )
