File: Battery_Charger.kicad_pcb (KiCad board)
At the start: 2 copper layers, 16.5 x 25.6 mm, 9 parts, among them J1 USB_B_Micro, J2 Conn_01x02, U1 MCP73831-2-OT

Commit message: ......
Routing:
- net GND: track 42.5 -> 44.0 mm
Changed lines of the file:
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@@
-	)
-	(segment
-		(start 147.475 78.9875)
-		(end 147.475 83.405)
-		(width 0.25)
-		(layer "F.Cu")
-		(net 2)
 	)
 	(segment
@@
 	)
 	(segment
+		(start 147.205 83.675)
+		(end 145.575 83.675)
+		(width 0.25)
+		(layer "F.Cu")
+		(net 2)
+	)
+	(segment
+		(start 144.6825 76.195)
+		(end 147.175 76.195)
+		(width 0.25)
+		(layer "F.Cu")
+		(net 2)
+	)
+	(segment
 		(start 142.345 73.225)
 		(end 144.6825 75.5625)
@@
 	)
 	(segment
-		(start 144.6825 76.195)
-		(end 147.475 78.9875)
+		(start 144.1225 83.675)
+		(end 142.8525 84.945)
 		(width 0.25)
 		(layer "F.Cu")
@@
 	)
 	(segment
-		(start 144.1225 83.675)
-		(end 142.8525 84.945)
+		(start 147.475 76.495)
+		(end 147.475 83.405)
 		(width 0.25)
 		(layer "F.Cu")
@@
 	)
 	(segment
-		(start 147.205 83.675)
-		(end 145.575 83.675)
+		(start 141.19 83.2825)
+		(end 142.8525 84.945)
 		(width 0.25)
 		(layer "F.Cu")
@@
 	)
 	(segment
-		(start 141.19 83.2825)
-		(end 142.8525 84.945)
+		(start 147.175 76.195)
+		(end 147.475 76.495)
 		(width 0.25)
 		(layer "F.Cu")
